Commit message: Changed mass of monoped base to match that of towr mass, still issues with final trajectory

File: rsc/monoped/monoped.urdf (robot description, URDF)
Before this commit: robot monoped, 4 links, 3 joints
Links:
- link base: mass 0.18 -> 20
- link lowerleg: mass 0.18 -> 0.2
- link upperleg: mass 0.18 -> 0.2

Commit message: force traking,Jacobian alterd to method 1,mass of links changed,collision bodies accurate

File: rsc/monoped/monoped.urdf (robot description, URDF)
Before this commit: robot monoped, 4 links, 3 joints
Links:
- link hipassembly: mass 0.18 -> 0.02
- link lowerleg: mass 0.2 -> 0.02; geometry collision cylinder length=0.315 radius=0.015; visual mesh filename=lowerleg.dae scale=1 1 1
- link upperleg: mass 0.2 -> 0.02; geometry collision box size=0.33 0.05 0.05; visual mesh filename=upperleg.dae scale=1 1 1

Commit message: Made changes to monoped urdf, to add better collision boxes

File: rsc/monoped/monoped.urdf (robot description, URDF)
Before this commit: robot monoped, 4 links, 3 joints
Links:
- added link foot, mass 0.01; collision sphere radius=0.03; visual sphere radius=0.03
Joints:
- added joint fl_joint: type fixed, parent lowerleg, child foot, origin xyz=0.000 0.00000 0.00000 rpy=0.0 0.0 0.0

Commit message: Removed limits on joint forces for monoped urdf

File: rsc/monoped/monoped.urdf (robot description, URDF)
Before this commit: robot monoped, 5 links, 4 joints
Joints:
- joint haa_joint: limit lower=-1.6 upper=1.6 effort=200 velocity=1.0 -> lower=-3.14 upper=3.14 effort=200 velocity=100.0
- joint hfe_joint: limit lower=-1.6 upper=1.6 effort=200 velocity=1.0 -> lower=-3.14 upper=3.14 effort=200 velocity=100.0
- joint kfe_joint: limit lower=-1.6 upper=1.6 effort=200 velocity=1.0 -> lower=-3.14 upper=3.14 effort=200 velocity=100.0
